File: Hardware/CALCKS/CALCKS.sch (KiCad schematic (older format))
At the start: 68 parts, among them J1 Conn_02x03_Counter_Clockwise, J2 USB_B_Micro, J3 Conn_01x01_Male, J4 Conn_01x01_Male, SW1 SW_Push_Dual, SW10 SW_Push_Dual, SW11 SW_Push_Dual, SW12 SW_Push_Dual, SW13 SW_Push_Dual, SW14 SW_Push_Dual, SW15 SW_Push_Dual, SW16 SW_Push_Dual, SW17 SW_Push_Dual, SW18 SW_Push_Dual, SW19 SW_Push_Dual, SW2 SW_Push_Dual, SW20 SW_Push_Dual, SW21 SW_Push_Dual, SW22 SW_Push_Dual, SW23 SW_Push_Dual, SW24 SW_Push_Dual, SW25 SW_Push_Dual, SW26 SW_Push_Dual, SW27 SW_Push_Dual, SW28 SW_Push_Dual, SW29 SW_Push_Dual, SW3 SW_Push_Dual, SW30 SW_Push_Dual, SW31 SW_Push_Dual, SW32 SW_Push_Dual, SW33 SW_Push_Dual, SW34 SW_Push_Dual, SW35 SW_Push_Dual, SW36 SW_Push_Dual, SW37 SW_Push_Dual, SW38 SW_Push_Dual, SW39 SW_Push_Dual, SW4 SW_Push_Dual, SW40 SW_Push_Dual, SW5 SW_Push_Dual, SW6 SW_Push_Dual, SW7 SW_Push_Dual, SW8 SW_Push_Dual, SW9 SW_Push_Dual, U1 ATmega1284-AU, U2 MCP73831-2-OT, U3 AT24CS64-SSHM, U4 74HC164, Y1 16MHz

Commit message: PCB routing
Parts:
- J3, J4: footprint TestPoint:TestPoint_Pad_D3.0mm -> Connector_Wire:SolderWirePad_1x01_Drill1.2mm
Connections:
- net +BATT: now reaches C2.2, D1.2 (A), J4.1 (Pin_1), U2.3 (VBAT)
- net GND renamed -BATT
- net -BATT: no longer C1.2, J2.5 (GND), R1.1, U2.2 (VSS)
- new net: C1.2, J2.5 (GND), R1.1, U2.2 (VSS)
Other:
- note added: "Current regulation:\n3.3k -> 303mA"
Changed lines of the file:
@@
 	1    0    0    -1
-$EndComp
-$Comp
-L Connector:Conn_01x01_Male J4
-U 1 1 5F203408
-P 3050 1200
-F 0 "J4" H 3022 1224 50  0000 R CNN
-F 1 "Conn_01x01_Male" H 3022 1133 50  0000 R CNN
-F 2 "TestPoint:TestPoint_Pad_D3.0mm" H 3050 1200 50  0001 C CNN
-F 3 "~" H 3050 1200 50  0001 C CNN
-	1    3050 1200
-	-1   0    0    -1
 $EndComp
 Wire Wire Line
@@
 	1600 1000 1700 1000
 $Comp
-L power:GND #PWR0102
-U 1 1 5F28F479
-P 1250 1700
-F 0 "#PWR0102" H 1250 1450 50  0001 C CNN
-F 1 "GND" H 1255 1527 50  0000 C CNN
-F 2 "" H 1250 1700 50  0001 C CNN
-F 3 "" H 1250 1700 50  0001 C CNN
-	1    1250 1700
-	1    0    0    -1
-$EndComp
-$Comp
-L Connector:Conn_01x01_Male J3
-U 1 1 5F29013F
-P 2300 1900
-F 0 "J3" V 2454 1812 50  0000 R CNN
-F 1 "Conn_01x01_Male" V 2363 1812 50  0000 R CNN
-F 2 "TestPoint:TestPoint_Pad_D3.0mm" H 2300 1900 50  0001 C CNN
-F 3 "~" H 2300 1900 50  0001 C CNN
-	1    2300 1900
-	0    -1   -1   0
-$EndComp
-$Comp
 L Device:C C1
 U 1 1 5F292FC0
@@
 Wire Wire Line
 	1600 1700 1250 1700
-Connection ~ 1250 1700
-Connection ~ 2300 1700
 $Comp
 L power:GND #PWR0103
@@
 	0    -1   -1   0
 $EndComp
-Connection ~ 2850 1200
 Wire Wire Line
 	2100 2800 2200 2800
@@
 Wire Wire Line
 	2850 1200 2850 1550
-Text GLabel 3150 1550 2    50   Input ~ 0
-VCC
 Text GLabel 6700 2450 2    50   Input ~ 0
 VCC
@@
 Wire Wire Line
 	9700 6300 11000 6300
+Text Notes 1500 1900 0    50   ~ 0
+Current regulation:\n3.3k -> 303mA
+Text GLabel 3150 1550 2    50   Input ~ 0
+VCC
+$Comp
+L power:+BATT #PWR0109
+U 1 1 5EF8C1E9
+P 3050 1200
+F 0 "#PWR0109" H 3050 1050 50  0001 C CNN
+F 1 "+BATT" V 3065 1328 50  0000 L CNN
+F 2 "" H 3050 1200 50  0001 C CNN
+F 3 "" H 3050 1200 50  0001 C CNN
+	1    3050 1200
+	0    1    1    0
+$EndComp
+Connection ~ 2850 1200
+Wire Wire Line
+	3050 1200 2850 1200
+$Comp
+L power:+BATT #PWR0111
+U 1 1 5EFF3135
+P 4650 1000
+F 0 "#PWR0111" H 4650 850 50  0001 C CNN
+F 1 "+BATT" H 4665 1173 50  0000 C CNN
+F 2 "" H 4650 1000 50  0001 C CNN
+F 3 "" H 4650 1000 50  0001 C CNN
+	1    4650 1000
+	1    0    0    -1
+$EndComp
+$Comp
+L power:-BATT #PWR0112
+U 1 1 5F053D34
+P 4400 1000
+F 0 "#PWR0112" H 4400 850 50  0001 C CNN
+F 1 "-BATT" H 4415 1173 50  0000 C CNN
+F 2 "" H 4400 1000 50  0001 C CNN
+F 3 "" H 4400 1000 50  0001 C CNN
+	1    4400 1000
+	1    0    0    -1
+$EndComp
+$Comp
+L Connector:Conn_01x01_Male J3
+U 1 1 5F055712
+P 4400 1200
+F 0 "J3" V 4450 1350 50  0000 R CNN
+F 1 "Conn_01x01_Male" V 4350 1800 50  0000 R CNN
+F 2 "Connector_Wire:SolderWirePad_1x01_Drill1.2mm" H 4400 1200 50  0001 C CNN
+F 3 "~" H 4400 1200 50  0001 C CNN
+	1    4400 1200
+	0    -1   -1   0
+$EndComp
+$Comp
+L Connector:Conn_01x01_Male J4
+U 1 1 5F218788
+P 4650 1200
+F 0 "J4" V 4800 1400 50  0000 R CNN
+F 1 "Conn_01x01_Male" V 4700 1900 50  0000 R CNN
+F 2 "Connector_Wire:SolderWirePad_1x01_Drill1.2mm" H 4650 1200 50  0001 C CNN
+F 3 "~" H 4650 1200 50  0001 C CNN
+	1    4650 1200
+	0    1    -1   0
+$EndComp
+$Comp
+L power:GND #PWR0102
+U 1 1 5F3257DD
+P 4400 1000
+F 0 "#PWR0102" H 4400 750 50  0001 C CNN
+F 1 "GND" H 4300 850 50  0000 C CNN
+F 2 "" H 4400 1000 50  0001 C CNN
+F 3 "" H 4400 1000 50  0001 C CNN
+	1    4400 1000
+	0    1    1    0
+$EndComp
+Connection ~ 4400 1000
 $EndSCHEMATC

Commit message: small changes
Parts:
- Y1: value 16MHz -> 8MHz
Changed lines of the file:
@@
 P 1250 3600
 F 0 "Y1" V 1300 3400 50  0000 L CNN
-F 1 "16MHz" V 1200 3200 50  0000 L CNN
+F 1 "8MHz" V 1200 3200 50  0000 L CNN
 F 2 "Crystal:Crystal_SMD_HC49-SD" H 1250 3600 50  0001 C CNN
 F 3 "~" H 1250 3600 50  0001 C CNN

Commit message: Final changes to PCB before sending it off
Parts:
- added C12, C13: 30pF, Capacitor_SMD:C_0805_2012Metric, symbol Device:C
Connections:
- net -BATT: now also C12.2, C13.1
- net at U1.7 (XTAL2), Y1.1: now also C13.2
- net at U1.8 (XTAL1), Y1.2: now also C12.1
Changed lines of the file:
@@
 VCC
-Wire Wire Line
-	2200 2800 2200 3000
 Wire Wire Line
 	2100 2800 2100 3000
@@
 Wire Wire Line
 	3950 4800 3950 5000
-Text GLabel 3500 5400 3    50   Input ~ 0
-VCC
 Wire Wire Line
 	3100 5000 3100 4800
@@
 Wire Wire Line
 	2700 1400 2700 1700
-Wire Wire Line
-	2700 1700 3050 1700
 Text GLabel 3050 1700 2    50   Input ~ 0
 BATT_STATUS
 Text GLabel 2700 4200 2    50   Input ~ 0
 BATT_STATUS
-$Comp
-L Device:Crystal Y1
-U 1 1 603ADCA6
-P 1250 3600
-F 0 "Y1" V 1300 3400 50  0000 L CNN
-F 1 "8MHz" V 1200 3200 50  0000 L CNN
-F 2 "Crystal:Crystal_SMD_HC49-SD" H 1250 3600 50  0001 C CNN
-F 3 "~" H 1250 3600 50  0001 C CNN
-	1    1250 3600
-	0    1    -1   0
-$EndComp
 Wire Wire Line
 	1250 3450 1450 3450
@@
 $EndComp
 Connection ~ 4400 1000
+$Comp
+L Device:Crystal Y1
+U 1 1 603ADCA6
+P 1250 3600
+F 0 "Y1" V 1300 3400 50  0000 L CNN
+F 1 "8MHz" V 1200 3200 50  0000 L CNN
+F 2 "Crystal:Crystal_SMD_HC49-SD" H 1250 3600 50  0001 C CNN
+F 3 "~" H 1250 3600 50  0001 C CNN
+	1    1250 3600
+	0    1    -1   0
+$EndComp
+$Comp
+L Device:C C13
+U 1 1 5EFDD062
+P 1100 3900
+F 0 "C13" H 986 3854 50  0000 R CNN
+F 1 "30pF" H 1050 4000 50  0000 R CNN
+F 2 "Capacitor_SMD:C_0805_2012Metric" H 1138 3750 50  0001 C CNN
+F 3 "~" H 1100 3900 50  0001 C CNN
+	1    1100 3900
+	1    0    0    1
+$EndComp
+Wire Wire Line
+	1250 3450 1100 3450
+Connection ~ 1250 3450
+Wire Wire Line
+	1250 3750 1100 3750
+Connection ~ 1250 3750
+Wire Wire Line
+	1100 3150 800  3150
+Wire Wire Line
+	800  3150 800  3600
+Wire Wire Line
+	800  4050 1100 4050
+$Comp
+L power:GND #PWR0110
+U 1 1 5F0676F1
+P 800 3600
+F 0 "#PWR0110" H 800 3350 50  0001 C CNN
+F 1 "GND" V 805 3472 50  0000 R CNN
+F 2 "" H 800 3600 50  0001 C CNN
+F 3 "" H 800 3600 50  0001 C CNN
+	1    800  3600
+	0    1    1    0
+$EndComp
+Connection ~ 800  3600
+Wire Wire Line
+	800  3600 800  4050
+Text GLabel 3500 5400 3    50   Input ~ 0
+VCC
+Wire Wire Line
+	2200 2800 2200 3000
+$Comp
+L Device:C C12
+U 1 1 5EFDC2E9
+P 1100 3300
+F 0 "C12" H 986 3254 50  0000 R CNN
+F 1 "30pF" H 1050 3400 50  0000 R CNN
+F 2 "Capacitor_SMD:C_0805_2012Metric" H 1138 3150 50  0001 C CNN
+F 3 "~" H 1100 3300 50  0001 C CNN
+	1    1100 3300
+	1    0    0    1
+$EndComp
+Wire Wire Line
+	2700 1700 3050 1700
 $EndSCHEMATC
