File: Hardware/CALCKS/CALCKS.sch (KiCad schematic (older format))
At the start: 70 parts, among them J1 Conn_02x03_Counter_Clockwise, J2 USB_B_Micro, J3 Conn_01x01_Male, J4 Conn_01x01_Male, SW1 SW_Push_Dual, SW10 SW_Push_Dual, SW11 SW_Push_Dual, SW12 SW_Push_Dual, SW13 SW_Push_Dual, SW14 SW_Push_Dual, SW15 SW_Push_Dual, SW16 SW_Push_Dual, SW17 SW_Push_Dual, SW18 SW_Push_Dual, SW19 SW_Push_Dual, SW2 SW_Push_Dual, SW20 SW_Push_Dual, SW21 SW_Push_Dual, SW22 SW_Push_Dual, SW23 SW_Push_Dual, SW24 SW_Push_Dual, SW25 SW_Push_Dual, SW26 SW_Push_Dual, SW27 SW_Push_Dual, SW28 SW_Push_Dual, SW29 SW_Push_Dual, SW3 SW_Push_Dual, SW30 SW_Push_Dual, SW31 SW_Push_Dual, SW32 SW_Push_Dual, SW33 SW_Push_Dual, SW34 SW_Push_Dual, SW35 SW_Push_Dual, SW36 SW_Push_Dual, SW37 SW_Push_Dual, SW38 SW_Push_Dual, SW39 SW_Push_Dual, SW4 SW_Push_Dual, SW40 SW_Push_Dual, SW5 SW_Push_Dual, SW6 SW_Push_Dual, SW7 SW_Push_Dual, SW8 SW_Push_Dual, SW9 SW_Push_Dual, U1 ATmega1284-AU, U2 MCP73831-2-OT, U3 AT24CS64-SSHM, U4 74HC164, Y1 8MHz

Commit message: Version 2 of PCB
Parts:
- added C17, C3, C5, C7: 0.1uF, Capacitor_SMD:C_0805_2012Metric, symbol Device:C
- added H1, H2, H3, H4, H5: MountingHole_Pad, MountingHole:MountingHole_2.2mm_M2_Pad_Via, symbol Mechanical:MountingHole_Pad
- added J5: Conn_01x04_Male, Connector_PinHeader_2.54mm:PinHeader_1x04_P2.54mm_Horizontal, symbol Connector:Conn_01x04_Male
- D1: footprint Diode_SMD:D_SOD-323 -> Diode_SMD:D_SOD-323_HandSoldering
- renumbered C12 to C1, C5 to C10, C6 to C11, C7 to C12, C8 to C13, C9 to C14, C10 to C15, C11 to C16, C13 to C2, C1 to C4, C2 to C6, C3 to C8, C4 to C9, J2 to J1, J1 to J2, R2 to R3, R3 to R4, R4 to R5, R5 to R6, R6 to R7, SW8 to SW1, SW5 to SW10, SW6 to SW11, SW7 to SW12, SW9 to SW13, SW10 to SW14, SW11 to SW15, SW12 to SW16, SW13 to SW17, SW14 to SW18, SW15 to SW19, SW16 to SW2, SW17 to SW20, SW18 to SW21, SW19 to SW22, SW20 to SW23, SW21 to SW24, SW22 to SW25, SW23 to SW26, SW25 to SW27, SW26 to SW28, SW27 to SW29, SW24 to SW3, SW28 to SW30, SW29 to SW31, SW30 to SW32, SW31 to SW33, SW33 to SW35, SW35 to SW36, SW36 to SW37, SW37 to SW38, SW38 to SW39, SW32 to SW4, SW39 to SW40, SW40 to SW5, SW1 to SW6, SW2 to SW7, SW3 to SW8, SW4 to SW9
Connections:
- net -BATT: now also SW1.4, SW2.4, SW3.4, SW4.4, SW5.4, C17.1, C3.1, C5.1, C7.1, H1.1, H2.1, H3.1, H4.1, H5.1, J5.1 (Pin_1)
- net BTN_ROW1: now also SW10.4, SW11.4, SW12.4, SW6.4, SW7.4, SW8.4, SW9.4, U1.11 (PD2); no longer SW1.2, SW10.2, SW11.2, SW12.2, SW6.2, SW7.2, SW8.2, SW9.2, U1.9 (PD0)
- net BTN_ROW2: now also SW13.4, SW14.4, SW15.4, SW16.4, SW17.4, SW18.4, SW19.4, U1.12 (PD3); no longer SW13.2, SW14.2, SW15.2, SW16.2, SW17.2, SW18.2, SW19.2, SW2.2, U1.10 (PD1)
- net BTN_ROW3: now also SW20.4, SW21.4, SW22.4, SW23.4, SW24.4, SW25.4, SW26.4, U1.13 (PD4); no longer SW20.2, SW21.2, SW22.2, SW23.2, SW24.2, SW25.2, SW26.2, SW3.2, U1.11 (PD2)
- net BTN_ROW4: now also SW27.4, SW28.4, SW29.4, SW30.4, SW31.4, SW32.4, SW33.4, U1.14 (PD5); no longer SW27.2, SW28.2, SW29.2, SW30.2, SW31.2, SW32.2, SW33.2, SW4.2, U1.12 (PD3)
- net BTN_ROW5: now also SW34.4, SW35.4, SW36.4, SW37.4, SW38.4, SW39.4, SW40.4, U1.15 (PD6); no longer SW34.2, SW35.2, SW36.2, SW37.2, SW38.2, SW39.2, SW40.2, SW5.2, U1.13 (PD4)
- net CLK: now also U1.41 (PB1); no longer U1.14 (PD5)
- net CLR: now also U1.42 (PB2); no longer U1.15 (PD6)
- net VCC: now also C17.2, C5.2, C7.2, J5.4 (Pin_4); no longer U1.29 (AREF)
- net at U1.21 (PC2): now also SW1.1
- net at U1.22 (PC3): now also SW2.1
- net at U1.23 (PC4): now also SW3.1
- net at U1.24 (PC5): now also SW4.1
- net at U1.25 (PC6): now also SW5.1
- new net: C3.2, U1.29 (AREF)
- new net RXD0: J5.3 (Pin_3), U1.9 (PD0)
- new net TXD0: J5.2 (Pin_2), U1.10 (PD1)
- now unconnected: U4.13 (Q7)
- no-connect marks 106 -> 100
Other:
- moved on the sheet: D1, J1, J4, R3, R4, R5, R6, R7, SW1, SW2, SW3, SW4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
