File: Hardware/CALCKS/CALCKS.kicad_pcb (KiCad board)
At the start: 2 copper layers, 68 parts, among them J1 Conn_02x03_Counter_Clockwise, J2 USB_B_Micro, J3 Conn_01x01_Male, J4 Conn_01x01_Male, SW1 SW_Push_Dual, SW10 SW_Push_Dual, SW11 SW_Push_Dual, SW12 SW_Push_Dual, SW13 SW_Push_Dual, SW14 SW_Push_Dual, SW15 SW_Push_Dual, SW16 SW_Push_Dual, SW17 SW_Push_Dual, SW18 SW_Push_Dual, SW19 SW_Push_Dual, SW2 SW_Push_Dual, SW20 SW_Push_Dual, SW21 SW_Push_Dual, SW22 SW_Push_Dual, SW23 SW_Push_Dual, SW24 SW_Push_Dual, SW25 SW_Push_Dual, SW26 SW_Push_Dual, SW27 SW_Push_Dual, SW28 SW_Push_Dual, SW29 SW_Push_Dual, SW3 SW_Push_Dual, SW30 SW_Push_Dual, SW31 SW_Push_Dual, SW32 SW_Push_Dual, SW33 SW_Push_Dual, SW34 SW_Push_Dual, SW35 SW_Push_Dual, SW36 SW_Push_Dual, SW37 SW_Push_Dual, SW38 SW_Push_Dual, SW39 SW_Push_Dual, SW4 SW_Push_Dual, SW40 SW_Push_Dual, SW5 SW_Push_Dual, SW6 SW_Push_Dual, SW7 SW_Push_Dual, SW8 SW_Push_Dual, SW9 SW_Push_Dual, U1 ATmega1284-AU, U2 MCP73831-2-OT, U3 AT24CS64-SSHM, U4 74HC164, Y1 16MHz

Commit message: PCB routing
Parts:
- C1, C10, C11, C3, C4, C5, C6, C7, C8, C9, D1: moved to B.Cu
- J3, J4: footprint TestPoint:TestPoint_Pad_D3.0mm -> Connector_Wire:SolderWirePad_1x01_Drill1.2mm
- moved D1 38.2 mm to (100.3, 50.8)
- moved U4 34.7 mm to (101.0, 113.7), turned to 270 degrees
- moved SW10 28.7 mm to (86.4, 113.7)
- moved J3 28.1 mm to (100.3, 88.3)
- moved J4 26.2 mm to (91.4, 88.3)
- moved C2 19.9 mm to (95.9, 88.3), turned to 180 degrees
- moved SW26 16.5 mm to (109.9, 97.2)
- moved C1 11.7 mm to (98.4, 34.3)
- moved U3 9.61 mm to (75.6, 104.8), turned to 0 degrees
- moved C10 7.65 mm to (73.7, 72.4), turned to 270 degrees
- moved C9 7.65 mm to (73.7, 64.8), turned to 90 degrees
- moved U1 7.01 mm to (94.6, 101.6)
- moved J1 4.49 mm to (75.6, 96.5), turned to 180 degrees
- moved R1 1.42 mm to (109.9, 28.6), turned to 180 degrees
- moved U2 0.90 mm to (106.0, 31.1)
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Connections:
- net Net-(C2-Pad2) renamed +BATT
- C1 pad 2: GND -> Net-(C1-Pad2)
- C10 pad 1: GND -> -BATT
- C11 pad 1: GND -> -BATT
- C2 pad 1: GND -> -BATT
- C3 pad 1: GND -> -BATT
- C5 pad 1: GND -> -BATT
- C6 pad 1: GND -> -BATT
- C9 pad 1: GND -> -BATT
- DS1 pad 26: GND -> -BATT
- DS1 pad 33: GND -> -BATT
- J1 pad 4: GND -> -BATT
- J2 pad 5: GND -> Net-(C1-Pad2)
- J3 pad 1: GND -> -BATT
- R1 pad 1: GND -> Net-(C1-Pad2)
- R2 pad 2: GND -> -BATT
- R3 pad 2: GND -> -BATT
- R4 pad 2: GND -> -BATT
- R5 pad 2: GND -> -BATT
- R6 pad 2: GND -> -BATT
- U1 pad 18: GND -> -BATT
- U1 pad 28: GND -> -BATT
- U1 pad 39: GND -> -BATT
- U1 pad 6: GND -> -BATT
- U2 pad 2: GND -> Net-(C1-Pad2)
- U3 pad 1: GND -> -BATT
- U3 pad 2: GND -> -BATT
- U3 pad 3: GND -> -BATT
- U3 pad 4: GND -> -BATT
- U3 pad 7: GND -> -BATT
- U4 pad 7: GND -> -BATT
Routing:
- net -BATT: track 0.00 -> 159.5 mm, vias 0 -> 6
- net BTN_ROW3: track 0.00 -> 151.0 mm, vias 0 -> 8
- net BTN_ROW4: track 0.00 -> 143.7 mm, vias 0 -> 11
- net BTN_ROW5: track 0.00 -> 142.7 mm, vias 0 -> 2
- net BTN_ROW2: track 0.00 -> 128.7 mm, vias 0 -> 9
- net BTN_ROW1: track 0.00 -> 122.9 mm, vias 0 -> 10
- net Net-(SW16-Pad1): track 0.00 -> 109.6 mm, vias 0 -> 2
- net Net-(SW15-Pad1): track 0.00 -> 100.7 mm, vias 0 -> 2
- net Net-(SW14-Pad1): track 0.00 -> 96.1 mm, vias 0 -> 2
- net Net-(SW1-Pad1): track 0.00 -> 90.0 mm, vias 0 -> 4
- net Net-(SW13-Pad1): track 0.00 -> 80.3 mm, vias 0 -> 2
- net SCK: track 0.00 -> 78.6 mm, vias 0 -> 3
- net Net-(SW12-Pad1): track 0.00 -> 75.7 mm, vias 0 -> 2
- net BATT_STATUS: track 0.00 -> 71.4 mm
- net Net-(SW10-Pad1): track 0.00 -> 70.8 mm, vias 0 -> 3
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- added copper zone on F.Cu, net -BATT
- added copper zone on B.Cu, net VCC
Other:
- board outline added: 62.9 x 153.7 mm
- board text added: "CALCKS Prototype 1"

Commit message: small changes
Parts:
- Y1: value 16MHz -> 8MHz
- moved R6 3.94 mm to (122.4, 177.0)
Routing:
- net -BATT: track 159.5 -> 107.8 mm
Other:
- board text added: "JLCJLCJLCJLC"
Changed lines of the file:
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@@
   (general
     (thickness 1.6)
-    (drawings 9)
-    (tracks 778)
+    (drawings 10)
+    (tracks 760)
     (zones 0)
     (modules 68)
@@
     (pad_drill 0)
     (pad_to_mask_clearance 0)
-    (aux_axis_origin 0 0)
+    (aux_axis_origin 100.838 113.538)
     (visible_elements 7FFFFFFF)
     (pcbplotparams
@@
   )
   (module Resistor_SMD:R_0805_2012Metric (layer F.Cu)
-    (at 126.365 177.165 180)
+    (at 122.428 177.038 180)
     (descr "Resistor SMD 0805 (2012 Metric), square (rectangular) end terminal, IPC_7351 nominal, (Body size source: https://docs.google.com/spreadsheets/d/1BsfQQcO9C6DZCsRaXUlFlo91Tg2WpOkGARC1WS5S8t0/edit?usp=sharing), generated with kicad-footprint-generator")
     (tags resistor)
@@
       (effects (font (size 1 1) (thickness 0.15)))
     )
-    (fp_text value 16MHz (at 0 3.55 90) (layer F.Fab)
+    (fp_text value 8MHz (at 0 3.55 90) (layer F.Fab)
       (effects (font (size 1 1) (thickness 0.15)))
     )
@@
       (net 149 +BATT))
   )
-  (gr_text "CALCKS Prototype 1" (at 80.264 29.718) (layer F.SilkS)
+  (gr_text JLCJLCJLCJLC (at 119.38 31.496) (layer F.Cu)
+    (effects (font (size 1.5 1.5) (thickness 0.3)))
+  )
+  (gr_text "CALCKS\nPrototype 1" (at 80.518 29.972) (layer F.SilkS)
     (effects (font (size 1.5 1.5) (thickness 0.3)))
   )
@@
   (segment (start 125.729999 159.115001) (end 125.729999 168.489999) (width 0.25) (layer F.Cu) (net 111))
   (segment (start 127.105 159.04) (end 125.805 159.04) (width 0.25) (layer F.Cu) (net 111))
-  (segment (start 126.816973 176.679473) (end 127.3025 177.165) (width 0.25) (layer F.Cu) (net 111))
-  (segment (start 125.729999 175.592499) (end 126.816973 176.679473) (width 0.25) (layer F.Cu) (net 111))
-  (segment (start 125.729999 168.640001) (end 125.729999 175.592499) (width 0.25) (layer F.Cu) (net 111))
-  (segment (start 125.805 168.565) (end 125.729999 168.640001) (width 0.25) (layer F.Cu) (net 111))
-  (segment (start 127.105 168.565) (end 125.805 168.565) (width 0.25) (layer F.Cu) (net 111))
   (via (at 117.565 88.265) (size 0.8) (drill 0.4) (layers F.Cu B.Cu) (net 111))
   (segment (start 120.12 87.92) (end 117.91 87.92) (width 0.25) (layer F.Cu) (net 111))
@@
   (segment (start 91.44 107.275) (end 91.415 107.3) (width 0.25) (layer F.Cu) (net 111))
   (segment (start 91.44 105.955) (end 91.44 107.275) (width 0.25) (layer F.Cu) (net 111))
+  (segment (start 125.805 168.565) (end 127.105 168.565) (width 0.25) (layer F.Cu) (net 111))
+  (segment (start 123.3655 171.0045) (end 125.805 168.565) (width 0.25) (layer F.Cu) (net 111))
+  (segment (start 123.3655 177.038) (end 123.3655 171.0045) (width 0.25) (layer F.Cu) (net 111))
   (segment (start 88.104998 102.4) (end 88.915 102.4) (width 0.25) (layer F.Cu) (net 124))
   (segment (start 83.240001 89.805001) (end 83.240001 97.535003) (width 0.25) (layer F.Cu) (net 124))
@@
   (segment (start 96.00999 92.70501) (end 93.815 94.9) (width 0.25) (layer F.Cu) (net 145))
   (segment (start 104.945 30.165) (end 105.435002 30.165) (width 0.25) (layer F.Cu) (net 145))
-  (segment (start 88.746973 177.650527) (end 89.2325 177.165) (width 0.25) (layer F.Cu) (net 148))
-  (segment (start 88.20749 178.19001) (end 88.746973 177.650527) (width 0.25) (layer F.Cu) (net 148))
-  (segment (start 78.19251 178.19001) (end 88.20749 178.19001) (width 0.25) (layer F.Cu) (net 148))
-  (segment (start 77.1675 177.165) (end 78.19251 178.19001) (width 0.25) (layer F.Cu) (net 148))
-  (segment (start 100.27249 178.19001) (end 100.811973 177.650527) (width 0.25) (layer F.Cu) (net 148))
-  (segment (start 90.25751 178.19001) (end 100.27249 178.19001) (width 0.25) (layer F.Cu) (net 148))
-  (segment (start 100.811973 177.650527) (end 101.2975 177.165) (width 0.25) (layer F.Cu) (net 148))
-  (segment (start 89.2325 177.165) (end 90.25751 178.19001) (width 0.25) (layer F.Cu) (net 148))
-  (segment (start 112.876973 177.650527) (end 113.3625 177.165) (width 0.25) (layer F.Cu) (net 148))
-  (segment (start 112.33749 178.19001) (end 112.876973 177.650527) (width 0.25) (layer F.Cu) (net 148))
-  (segment (start 102.32251 178.19001) (end 112.33749 178.19001) (width 0.25) (layer F.Cu) (net 148))
-  (segment (start 101.2975 177.165) (end 102.32251 178.19001) (width 0.25) (layer F.Cu) (net 148))
-  (segment (start 124.941973 177.650527) (end 125.4275 177.165) (width 0.25) (layer F.Cu) (net 148))
-  (segment (start 114.38751 178.19001) (end 124.40249 178.19001) (width 0.25) (layer F.Cu) (net 148))
-  (segment (start 124.40249 178.19001) (end 124.941973 177.650527) (width 0.25) (layer F.Cu) (net 148))
-  (segment (start 113.3625 177.165) (end 114.38751 178.19001) (width 0.25) (layer F.Cu) (net 148))
   (segment (start 84.7575 74.2675) (end 86.995 76.505) (width 0.25) (layer B.Cu) (net 148))
   (segment (start 84.7575 73.025) (end 84.7575 74.2675) (width 0.25) (layer B.Cu) (net 148))

Commit message: Final changes to PCB before sending it off
Parts:
- added C12: 30pF, Capacitor_SMD:C_0805_2012Metric, F.Cu at (77.5, 100.3)
- added C13: 30pF, Capacitor_SMD:C_0805_2012Metric, F.Cu at (73.0, 87.0)
- added G***: LOGO, CALCKS:kzo_logo, F.Cu at (120.7, 114.3)
- added MH1: MountingHole_2.2mm_M2_Pad, MountingHole:MountingHole_2.2mm_M2_Pad, F.Cu at (125.7, 29.8)
- added MH1: MountingHole_2.2mm_M2_Pad, MountingHole:MountingHole_2.2mm_M2_Pad, F.Cu at (70.5, 29.8)
- added MH3: MountingHole_2.2mm_M2_Pad, MountingHole:MountingHole_2.2mm_M2_Pad, F.Cu at (125.1, 106.0)
- added MH4: MountingHole_2.2mm_M2_Pad, MountingHole:MountingHole_2.2mm_M2_Pad, F.Cu at (69.8, 176.5)
- added MH5: MountingHole_2.2mm_M2_Pad, MountingHole:MountingHole_2.2mm_M2_Pad, F.Cu at (126.4, 176.5)
- moved C1 3.18 mm to (98.4, 37.5)
- moved R6 1.14 mm to (121.3, 177.0)
Routing:
- net Net-(C13-Pad2): track 16.8 -> 25.7 mm, vias 0 -> 2
- net Net-(C12-Pad1): track 9.06 -> 15.3 mm
- net Net-(C1-Pad2): track 22.1 -> 25.3 mm
- net Net-(C1-Pad1): track 13.8 -> 17.0 mm
- net -BATT: track 107.8 -> 106.9 mm

Commit message: Version 2 of PCB
Parts:
- removed MH1 (x2), MH3, MH4, MH5: MountingHole_2.2mm_M2_Pad, MountingHole:MountingHole_2.2mm_M2_Pad
- added C17: 0.1uF, Capacitor_SMD:C_0805_2012Metric, F.Cu at (111.8, 113.7)
- added C3: 0.1uF, Capacitor_SMD:C_0805_2012Metric, F.Cu at (103.5, 101.0)
- added C5: 0.1uF, Capacitor_SMD:C_0805_2012Metric, F.Cu at (97.2, 93.3)
- added C7: 0.1uF, Capacitor_SMD:C_0805_2012Metric, F.Cu at (81.3, 103.5)
- added H1: MountingHole_Pad, MountingHole:MountingHole_2.2mm_M2_Pad_Via, F.Cu at (69.8, 29.2)
- added H2: MountingHole_Pad, MountingHole:MountingHole_2.2mm_M2_Pad_Via, F.Cu at (126.4, 29.2)
- added H3: MountingHole_Pad, MountingHole:MountingHole_2.2mm_M2_Pad_Via, F.Cu at (126.4, 87.6)
- added H4: MountingHole_Pad, MountingHole:MountingHole_2.2mm_M2_Pad_Via, F.Cu at (69.6, 176.8)
- added H5: MountingHole_Pad, MountingHole:MountingHole_2.2mm_M2_Pad_Via, F.Cu at (126.7, 176.8)
- added J5: Conn_01x04_Male, Connector_PinHeader_2.54mm:PinHeader_1x04_P2.54mm_Horizontal, F.Cu at (76.2, 30.5)
- D1: footprint Diode_SMD:D_SOD-323 -> Diode_SMD:D_SOD-323_HandSoldering
- moved SW2 85.8 mm to (117.5, 90.8)
- moved SW3 74.1 mm to (111.3, 97.8)
- moved SW4 74.1 mm to (123.2, 97.8)
- moved SW5 66.2 mm to (117.5, 104.8)
- moved SW34 38.8 mm to (86.4, 112.6)
- moved SW35 32.8 mm to (122.6, 122.2)
- moved SW28 25.0 mm to (110.5, 122.2)
- moved SW21 24.9 mm to (98.4, 122.2)
- moved SW14 8.51 mm to (86.4, 122.2)
- moved SW15 8.38 mm to (86.4, 131.6)
- moved SW16 8.38 mm to (86.4, 141.1)
- moved SW17 8.38 mm to (86.4, 150.6)
- moved SW18 8.38 mm to (86.4, 160.1)
- moved SW19 8.38 mm to (86.4, 169.7)
- moved SW22 8.38 mm to (98.4, 131.6)
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- renumbered C12 to C1, C5 to C10, C6 to C11, C7 to C12, C8 to C13, C9 to C14, C10 to C15, C11 to C16, C13 to C2, C1 to C4, C2 to C6, C3 to C8, C4 to C9, J2 to J1, J1 to J2, R2 to R3, R3 to R4, R4 to R5, R5 to R6, R6 to R7, SW8 to SW1, SW5 to SW10, SW6 to SW11, SW7 to SW12, SW9 to SW13, SW10 to SW14, SW11 to SW15, SW12 to SW16, SW13 to SW17, SW14 to SW18, SW15 to SW19, SW16 to SW2, SW17 to SW20, SW18 to SW21, SW19 to SW22, SW20 to SW23, SW21 to SW24, SW22 to SW25, SW23 to SW26, SW25 to SW27, SW26 to SW28, SW27 to SW29, SW24 to SW3, SW28 to SW30, SW29 to SW31, SW30 to SW32, SW31 to SW33, SW33 to SW35, SW35 to SW36, SW36 to SW37, SW37 to SW38, SW38 to SW39, SW32 to SW4, SW39 to SW40, SW40 to SW5, SW1 to SW6, SW2 to SW7, SW3 to SW8, SW4 to SW9
Connections:
- SW1 pad 1: Net-(SW16-Pad1) (its old number) -> Net-(SW1-Pad1)
- SW1 pad 2: BTN_ROW1 -> Net-(SW1-Pad2)
- SW1 pad 4: Net-(SW8-Pad4) -> -BATT
- SW10 pad 2: BTN_ROW1 -> Net-(SW10-Pad2)
- SW10 pad 4: Net-(SW5-Pad4) -> BTN_ROW1
- SW11 pad 2: BTN_ROW1 -> Net-(SW11-Pad2)
- SW11 pad 4: Net-(SW6-Pad4) -> BTN_ROW1
- SW12 pad 2: BTN_ROW1 -> Net-(SW12-Pad2)
- SW12 pad 4: Net-(SW7-Pad4) -> BTN_ROW1
- SW13 pad 2: BTN_ROW2 -> Net-(SW13-Pad2)
- SW13 pad 4: Net-(SW9-Pad4) -> BTN_ROW2
- SW14 pad 2: BTN_ROW2 -> Net-(SW14-Pad2)
- SW14 pad 4: Net-(SW10-Pad4) -> BTN_ROW2
- SW15 pad 2: BTN_ROW2 -> Net-(SW15-Pad2)
- SW15 pad 4: Net-(SW11-Pad4) -> BTN_ROW2
- SW16 pad 2: BTN_ROW2 -> Net-(SW16-Pad2)
- SW16 pad 4: Net-(SW12-Pad4) -> BTN_ROW2
- SW17 pad 2: BTN_ROW2 -> Net-(SW17-Pad2)
- SW17 pad 4: Net-(SW13-Pad4) -> BTN_ROW2
- SW18 pad 2: BTN_ROW2 -> Net-(SW18-Pad2)
- SW18 pad 4: Net-(SW14-Pad4) -> BTN_ROW2
- SW19 pad 2: BTN_ROW2 -> Net-(SW19-Pad2)
- SW19 pad 4: Net-(SW15-Pad4) -> BTN_ROW2
- SW2 pad 1: Net-(SW16-Pad1) (its old number) -> Net-(SW2-Pad1)
- SW2 pad 2: BTN_ROW2 -> Net-(SW2-Pad2)
- SW2 pad 4: Net-(SW16-Pad4) -> -BATT
- SW20 pad 2: BTN_ROW3 -> Net-(SW20-Pad2)
- SW20 pad 4: Net-(SW17-Pad4) -> BTN_ROW3
- SW21 pad 2: BTN_ROW3 -> Net-(SW21-Pad2)
- SW21 pad 4: Net-(SW18-Pad4) -> BTN_ROW3
- SW22 pad 2: BTN_ROW3 -> Net-(SW22-Pad2)
- SW22 pad 4: Net-(SW19-Pad4) -> BTN_ROW3
- SW23 pad 2: BTN_ROW3 -> Net-(SW23-Pad2)
- SW23 pad 4: Net-(SW20-Pad4) -> BTN_ROW3
- SW24 pad 2: BTN_ROW3 -> Net-(SW24-Pad2)
- SW24 pad 4: Net-(SW21-Pad4) -> BTN_ROW3
- SW25 pad 2: BTN_ROW3 -> Net-(SW25-Pad2)
- SW25 pad 4: Net-(SW22-Pad4) -> BTN_ROW3
- SW26 pad 2: BTN_ROW3 -> Net-(SW26-Pad2)
- SW26 pad 4: Net-(SW23-Pad4) -> BTN_ROW3
- SW27 pad 2: BTN_ROW4 -> Net-(SW27-Pad2)
- SW27 pad 4: Net-(SW25-Pad4) -> BTN_ROW4
- SW28 pad 2: BTN_ROW4 -> Net-(SW28-Pad2)
- SW28 pad 4: Net-(SW26-Pad4) -> BTN_ROW4
- SW29 pad 2: BTN_ROW4 -> Net-(SW29-Pad2)
- SW29 pad 4: Net-(SW27-Pad4) -> BTN_ROW4
- SW3 pad 1: Net-(SW16-Pad1) (its old number) -> Net-(SW3-Pad1)
- SW3 pad 2: BTN_ROW3 -> Net-(SW3-Pad2)
- SW3 pad 4: Net-(SW24-Pad4) -> -BATT
- SW30 pad 2: BTN_ROW4 -> Net-(SW30-Pad2)
- SW30 pad 4: Net-(SW28-Pad4) -> BTN_ROW4
- SW31 pad 2: BTN_ROW4 -> Net-(SW31-Pad2)
- SW31 pad 4: Net-(SW29-Pad4) -> BTN_ROW4
- SW32 pad 2: BTN_ROW4 -> Net-(SW32-Pad2)
- SW32 pad 4: Net-(SW30-Pad4) -> BTN_ROW4
- SW33 pad 2: BTN_ROW4 -> Net-(SW33-Pad2)
- SW33 pad 4: Net-(SW31-Pad4) -> BTN_ROW4
- SW34 pad 2: BTN_ROW5 -> Net-(SW34-Pad2)
- SW34 pad 4: Net-(SW34-Pad4) -> BTN_ROW5
- SW35 pad 2: BTN_ROW5 -> Net-(SW35-Pad2)
- SW35 pad 4: Net-(SW33-Pad4) -> BTN_ROW5
- SW36 pad 2: BTN_ROW5 -> Net-(SW36-Pad2)
- SW36 pad 4: Net-(SW35-Pad4) -> BTN_ROW5
- SW37 pad 2: BTN_ROW5 -> Net-(SW37-Pad2)
- SW37 pad 4: Net-(SW36-Pad4) -> BTN_ROW5
- SW38 pad 2: BTN_ROW5 -> Net-(SW38-Pad2)
- SW38 pad 4: Net-(SW37-Pad4) -> BTN_ROW5
- SW39 pad 2: BTN_ROW5 -> Net-(SW39-Pad2)
- SW39 pad 4: Net-(SW38-Pad4) -> BTN_ROW5
- SW4 pad 1: Net-(SW16-Pad1) (its old number) -> Net-(SW4-Pad1)
- SW4 pad 2: BTN_ROW4 -> Net-(SW4-Pad2)
- SW4 pad 4: Net-(SW32-Pad4) -> -BATT
- SW40 pad 2: BTN_ROW5 -> Net-(SW40-Pad2)
- SW40 pad 4: Net-(SW39-Pad4) -> BTN_ROW5
- SW5 pad 1: Net-(SW16-Pad1) (its old number) -> Net-(SW5-Pad1)
- SW5 pad 2: BTN_ROW5 -> Net-(SW5-Pad2)
- SW5 pad 4: Net-(SW40-Pad4) -> -BATT
- SW6 pad 2: BTN_ROW1 -> Net-(SW6-Pad2)
- SW6 pad 4: Net-(SW1-Pad4) -> BTN_ROW1
- SW7 pad 2: BTN_ROW1 -> Net-(SW7-Pad2)
- SW7 pad 4: Net-(SW2-Pad4) -> BTN_ROW1
- SW8 pad 2: BTN_ROW1 -> Net-(SW8-Pad2)
- SW8 pad 4: Net-(SW3-Pad4) -> BTN_ROW1
- SW9 pad 2: BTN_ROW1 -> Net-(SW9-Pad2)
- SW9 pad 4: Net-(SW4-Pad4) -> BTN_ROW1
- U1 pad 10: BTN_ROW2 -> TXD0
- U1 pad 11: BTN_ROW3 -> BTN_ROW1
- U1 pad 12: BTN_ROW4 -> BTN_ROW2
- U1 pad 13: BTN_ROW5 -> BTN_ROW3
- U1 pad 14: CLK -> BTN_ROW4
- U1 pad 15: CLR -> BTN_ROW5
- U1 pad 21: Net-(U1-Pad21) -> Net-(SW1-Pad1)
- U1 pad 22: Net-(U1-Pad22) -> Net-(SW2-Pad1)
- U1 pad 23: Net-(U1-Pad23) -> Net-(SW3-Pad1)
- U1 pad 24: Net-(U1-Pad24) -> Net-(SW4-Pad1)
- U1 pad 25: Net-(U1-Pad25) -> Net-(SW5-Pad1)
- U1 pad 29: VCC -> Net-(C3-Pad2)
- U1 pad 41: Net-(U1-Pad41) -> CLK
- U1 pad 42: Net-(U1-Pad42) -> CLR
- U1 pad 9: BTN_ROW1 -> RXD0
- U4 pad 13: Net-(SW16-Pad1) (its old number) -> Net-(U4-Pad13)
Routing:
- net Net-(SW14-Pad1): track 70.8 -> 199.1 mm, vias 3 -> 4
- net RXD0: track 0.00 -> 112.2 mm, vias 0 -> 1
- net Net-(SW16-Pad1) (its old number): track 109.6 -> 0.00 mm, vias 2 -> 0
- net TXD0: track 0.00 -> 102.3 mm, vias 0 -> 1
- net Net-(SW1-Pad1): track 0.00 -> 78.8 mm, vias 0 -> 2
- net VCC: track 38.6 -> 72.1 mm, vias 7 -> 9
- net Net-(SW13-Pad1): track 90.0 -> 123.0 mm, vias 4 -> 6
- net CLR: track 11.1 -> 41.8 mm, vias 0 -> 6
- net BTN_ROW5: track 143.4 -> 113.3 mm, vias 2 -> 0
- net Net-(SW16-Pad1): track 75.7 -> 104.8 mm, vias 2 -> 6
- net Net-(SW2-Pad1): track 0.00 -> 27.8 mm
- net Net-(SW4-Pad1): track 0.00 -> 25.2 mm
- net Net-(SW3-Pad1): track 0.00 -> 24.0 mm, vias 0 -> 2
- net SCK: track 78.6 -> 59.5 mm, vias 3 -> 1
- net Net-(SW15-Pad1): track 67.7 -> 85.9 mm, vias 2 -> 7
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Other:
- board text added: "CALCKS"
- board text removed: "CALCKS Prototype 1"
